File: LVDS_BeagleVFire_Cape.kicad_sch (KiCad schematic)
At the start: 3 parts, among them J8 Conn_01x06_Pin, P1 BeagleBone_Black_Header, P2 BeagleBone_Black_Header

Commit message: v2
Parts:
- added J9: ~, Kria_Board_Parts:LD3007MS_FAN, symbol Kria_Board_Parts:LD3007MS_FAN
Connections:
- net +5V: now also J9.2 (Fan+)
- net GND: now also J9.1 (Fan-)
