File: discriminator_inputs.kicad_sch (KiCad schematic)
At the start: 0 parts

Commit message: v2
Other:
- sheet Port A: file lvds_port.kicad_sch -> lvds_port_a.kicad_sch
- sheet Port A ports: added EN; removed none
- sheet Port B: file lvds_port.kicad_sch -> lvds_port_b.kicad_sch
- sheet Port B ports: added EN; removed none
Changed lines of the file:
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@@
 	(title_block
 		(title "BeagleV Fire TDC Cape")
-		(date "2024-09-28")
-		(rev "1")
+		(date "2025-01-31")
+		(rev "2")
 		(company "MIT SpinQuest DAQ Group")
 		(comment 1 "Noah Paladino")
+	)
+	(junction
+		(at 44.45 50.8)
+		(diameter 0)
+		(color 0 0 0 0)
 	)
 	(junction
@@
 	(wire
 		(pts
+			(xy 52.07 69.85) (xy 44.45 69.85)
+		)
+		(stroke
+			(width 0)
+			(type default)
+		)
+	)
+	(wire
+		(pts
 			(xy 52.07 67.31) (xy 35.56 67.31)
 		)
@@
 	(wire
 		(pts
+			(xy 44.45 43.18) (xy 44.45 50.8)
+		)
+		(stroke
+			(width 0)
+			(type default)
+		)
+	)
+	(wire
+		(pts
 			(xy 52.07 48.26) (xy 35.56 48.26)
 		)
@@
 		(pts
 			(xy 77.47 48.26) (xy 90.17 48.26)
+		)
+		(stroke
+			(width 0)
+			(type default)
+		)
+	)
+	(wire
+		(pts
+			(xy 44.45 69.85) (xy 44.45 50.8)
+		)
+		(stroke
+			(width 0)
+			(type default)
+		)
+	)
+	(wire
+		(pts
+			(xy 44.45 50.8) (xy 52.07 50.8)
 		)
 		(stroke
@@
 			)
 			(justify left bottom)
+		)
+	)
+	(global_label "~{SYS_RESET}"
+		(shape input)
+		(at 44.45 43.18 90)
+		(fields_autoplaced yes)
+		(effects
+			(font
+				(size 1.27 1.27)
+			)
+			(justify left)
+		)
+		(property "Intersheetrefs" "${INTERSHEET_REFS}"
+			(at 44.45 29.8794 90)
+			(effects
+				(font
+					(size 1.27 1.27)
+				)
+				(justify left)
+				(hide yes)
+			)
 		)
 	)
@@
 			)
 		)
-		(property "Sheetfile" "lvds_port.kicad_sch"
+		(property "Sheetfile" "lvds_port_b.kicad_sch"
 			(at 52.07 74.2446 0)
 			(effects
@@
 		(pin "VCC" input
 			(at 52.07 67.31 180)
+			(effects
+				(font
+					(size 1.27 1.27)
+				)
+				(justify left)
+			)
+		)
+		(pin "EN" input
+			(at 52.07 69.85 180)
 			(effects
 				(font
@@
 			)
 		)
-		(property "Sheetfile" "lvds_port.kicad_sch"
+		(property "Sheetfile" "lvds_port_a.kicad_sch"
 			(at 52.07 55.1946 0)
 			(effects
@@
 			(effects
 				(font
+					(size 1.27 1.27)
+				)
+				(justify left)
+			)
+		)
+		(pin "EN" input
+			(at 52.07 50.8 180)
+			(effects
+				(font
