File: lvds_port_b.kicad_sch (KiCad schematic)
At the start: 9 parts, among them J2 Conn_02x16, U5 SN65LVDT348D, U6 SN65LVDT348D, U7 SN65LVDT348D, U8 SN65LVDT348D

Commit message: v2
Parts:
- removed J2: Conn_02x16, Connector_PinHeader_2.54mm:PinHeader_2x16_P2.54mm_Vertical, symbol Connector_Generic:Conn_02x16_Odd_Even
- added J2: Conn_02x16, Kria_Board_Parts:PinHeader_2x17_P2.54mm_Vertical_ECL, symbol Connector_Generic:Conn_02x17_Odd_Even
- renumbered C5 to C1, C6 to C2, C7 to C3, C8 to C4, U5 to U1, U6 to U2, U7 to U3, U8 to U4
Connections:
- net In0+: now also J2.31 (Pin_31)
- net In0-: now also J2.32 (Pin_32)
- net In1+: now also J2.29 (Pin_29)
- net In1-: now also J2.30 (Pin_30)
- net In10+: now also J2.11 (Pin_11)
- net In10-: now also J2.12 (Pin_12)
- net In11+: now also J2.9 (Pin_9)
- net In11-: now also J2.10 (Pin_10)
- net In12+: now also J2.7 (Pin_7)
- net In12-: now also J2.8 (Pin_8)
- net In13+: now also J2.5 (Pin_5)
- net In13-: now also J2.6 (Pin_6)
- net In14+: now also J2.3 (Pin_3)
- net In14-: now also J2.4 (Pin_4)
- net In15+: now also J2.1 (Pin_1)
- net In15-: now also J2.2 (Pin_2)
- net In2+: now also J2.27 (Pin_27)
- net In2-: now also J2.28 (Pin_28)
- net In3+: now also J2.25 (Pin_25)
- net In3-: now also J2.26 (Pin_26)
- net In4+: now also J2.23 (Pin_23)
- net In4-: now also J2.24 (Pin_24)
- net In5+: now also J2.21 (Pin_21)
- net In5-: now also J2.22 (Pin_22)
- net In6+: now also J2.19 (Pin_19)
- net In6-: now also J2.20 (Pin_20)
- net In7+: now also J2.17 (Pin_17)
- net In7-: now also J2.18 (Pin_18)
- net In8+: now also J2.15 (Pin_15)
- net In8-: now also J2.16 (Pin_16)
- net In9+: now also J2.13 (Pin_13)
- net In9-: now also J2.14 (Pin_14)
- net Out0: now also U4.10 (ROUT4); no longer U1.15 (ROUT1)
- net Out1: now also U4.11 (ROUT3); no longer U1.14 (ROUT2)
- net Out10: now also U2.14 (ROUT2); no longer U3.11 (ROUT3)
- net Out11: now also U2.15 (ROUT1); no longer U3.10 (ROUT4)
- net Out12: now also U1.10 (ROUT4); no longer U4.15 (ROUT1)
- net Out13: now also U1.11 (ROUT3); no longer U4.14 (ROUT2)
- net Out14: now also U1.14 (ROUT2); no longer U4.11 (ROUT3)
- net Out15: now also U1.15 (ROUT1); no longer U4.10 (ROUT4)
- net Out2: now also U4.14 (ROUT2); no longer U1.11 (ROUT3)
- net Out3: now also U4.15 (ROUT1); no longer U1.10 (ROUT4)
- net Out4: now also U3.10 (ROUT4); no longer U2.15 (ROUT1)
- net Out5: now also U3.11 (ROUT3); no longer U2.14 (ROUT2)
- net Out6: now also U3.14 (ROUT2); no longer U2.11 (ROUT3)
- net Out7: now also U3.15 (ROUT1); no longer U2.10 (ROUT4)
- net Out8: now also U2.10 (ROUT4); no longer U3.15 (ROUT1)
- net Out9: now also U2.11 (ROUT3); no longer U3.14 (ROUT2)
- net VCC: no longer U1.16 (EN), U2.16 (EN), U3.16 (EN), U4.16 (EN)
- new net EN: U1.16 (EN), U2.16 (EN), U3.16 (EN), U4.16 (EN)
- no-connect marks 0 -> 2
